File: plate-pcb/su120-plate.kicad_pcb (KiCad board)
At the start: 2 copper layers, 98.8 x 98 mm, 194 parts, among them SW5 SW_Push

Commit message: Rev.2
Parts:
- removed the ? at (77.8, 116.7)
- removed the ? at (82.5, 116.7)
- removed the ? at (96.8, 116.7)
- removed the ? at (101.6, 116.7)
- removed the ? at (115.9, 116.7)
- removed the ? at (120.7, 116.7)
- removed the ? at (134.9, 116.7)
- removed the ? at (134.9, 131.0)
- removed the ? at (120.7, 131.0)
- removed the ? at (115.9, 131.0)
- removed the ? at (101.6, 131.0)
- removed the ? at (96.8, 131.0)
- removed the ? at (82.5, 131.0)
- removed the ? at (77.8, 131.0)
- removed the ? at (63.5, 131.0)
- removed the ? at (58.7, 131.0)
- removed the ? at (44.5, 131.0)
- removed the ? at (63.5, 135.7)
- removed the ? at (73.0, 135.7)
- removed the ? at (87.3, 135.7)
- removed the ? at (96.8, 135.7)
- removed the ? at (101.6, 135.7)
- removed the ? at (115.9, 135.7)
- removed the ? at (120.7, 135.7)
- removed the ? at (134.9, 135.7)
- removed the ? at (134.9, 150.0)
- removed the ? at (120.7, 150.0)
- removed the ? at (115.9, 150.0)
- removed the ? at (101.6, 150.0)
- removed the ? at (96.8, 150.0)
- removed the ? at (87.3, 150.0)
- removed the ? at (73.0, 150.0)
- removed the ? at (63.5, 150.0)
- removed the ? at (44.5, 59.5)
- removed the ? at (96.8, 59.5)
- removed the ? at (101.6, 59.5)
- removed the ? at (115.9, 59.5)
- removed the ? at (120.7, 59.5)
- removed the ? at (134.9, 59.5)
- removed the ? at (134.9, 73.8)
- removed the ? at (120.7, 73.8)
- removed the ? at (115.9, 73.8)
- removed the ? at (96.8, 73.8)
- removed the ? at (101.6, 73.8)
- removed the ? at (44.5, 73.8)
- removed the ? at (44.5, 78.6)
- removed the ? at (58.7, 78.6)
- removed the ? at (63.5, 78.6)
- removed the ? at (77.8, 78.6)
- removed the ? at (82.5, 78.6)
- removed the ? at (96.8, 78.6)
- removed the ? at (101.6, 78.6)
- removed the ? at (115.9, 78.6)
- removed the ? at (120.7, 78.6)
- removed the ? at (134.9, 78.6)
- removed the ? at (134.9, 92.9)
- removed the ? at (120.7, 92.9)
- removed the ? at (115.9, 92.9)
- removed the ? at (101.6, 92.9)
- removed the ? at (96.8, 92.9)
- removed the ? at (82.5, 92.9)
- removed the ? at (77.8, 92.9)
- removed the ? at (63.5, 92.9)
- removed the ? at (58.7, 92.9)
- removed the ? at (44.5, 92.9)
- removed the ? at (44.5, 97.6)
- removed the ? at (58.7, 97.6)
- removed the ? at (63.5, 97.6)
- removed the ? at (77.8, 97.6)
- removed the ? at (82.5, 97.6)
- removed the ? at (96.8, 97.6)
- removed the ? at (101.6, 97.6)
- removed the ? at (115.9, 97.6)
- removed the ? at (120.7, 97.6)
- removed the ? at (134.9, 97.6)
- removed the ? at (134.9, 111.9)
- removed the ? at (120.7, 111.9)
- removed the ? at (115.9, 111.9)
- removed the ? at (101.6, 111.9)
- removed the ? at (96.8, 111.9)
- removed the ? at (82.5, 111.9)
- removed the ? at (77.8, 111.9)
- removed the ? at (63.5, 111.9)
- removed the ? at (58.7, 111.9)
- removed the ? at (44.5, 111.9)
- removed the ? at (44.5, 116.7)
- removed the ? at (58.7, 116.7)
- removed the ? at (63.5, 116.7)
- SW5 (x2): footprint #footprint:Keyswitch_Plate_Hole -> #footprint:RotaryEncoder_Plate_Hole
Other:
- outline, holes or cut-outs redrawn
- board text removed: "A"
